File: lightstick_v4/lightstick_v4.kicad_pcb (KiCad board)
At the start: 4 copper layers, 43.1 x 66.5 mm, 78 parts, among them J1 FTSH-105-01-F-DV-P-TR, J2 USB_C_Receptacle, J3 Conn_01x03, J4 Conn_01x04, J5 2337019-1, J6 Conn_01x02, Q1 Q_NMOS_GSD, Q2 Q_NMOS_GSD, Q3 DMG2301L, SW1 SW_Push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

Commit message: rev1
Parts:
- removed J5: 2337019-1, Personal:TE_2337019-1
- added C30: C, Capacitor_SMD:C_0402_1005Metric, F.Cu at (100.5, 99.0)
- added J7: Conn_01x04, Connector_PinHeader_2.54mm:PinHeader_1x04_P2.54mm_Vertical, F.Cu at (68.9, 104.5)
- added L2: 2.2nH, Capacitor_SMD:C_0402_1005Metric, F.Cu at (99.0, 99.5)
- moved G*** 45.9 mm to (106.0, 136.7)
- moved J3 2.58 mm to (74.9, 85.4)
- moved C3 2.29 mm to (80.5, 99.4)
- moved R12 1.58 mm to (80.2, 96.3)
- moved R11 1.58 mm to (78.5, 96.3)
- moved Y2 1.01 mm to (83.1, 99.6), turned to 0 degrees
- moved C11 0.90 mm to (83.8, 96.4)
- moved C16 0.90 mm to (84.3, 97.7)
- moved C25 0.71 mm to (75.0, 91.9), turned to 0 degrees
- moved C4 0.60 mm to (83.8, 101.3)
- moved C5 0.56 mm to (97.5, 99.0)
- moved C6 0.56 mm to (94.5, 99.0)
- moved L1 0.51 mm to (96.0, 99.5)
- moved AE1 0.40 mm to (106.1, 98.8)
Connections:
- C5 pad 1: Net-(AE1-Pad1) -> Net-(C5-Pad1)
- L1 pad 1: Net-(AE1-Pad1) -> Net-(C5-Pad1)
- U1 pad P2: unconnected-(U1-P1.08-PadP2) -> Net-(J7-Pin_2)
- U1 pad R1: unconnected-(U1-TRACEDATA3/P1.09-PadR1) -> Net-(J7-Pin_3)
Routing:
- net Net-(J7-Pin_2): track 0.00 -> 18.0 mm, vias 0 -> 1
- net Net-(J7-Pin_3): track 0.00 -> 14.2 mm
- net GND: track 69.7 -> 75.2 mm, vias 86 -> 216
- net LED: track 20.8 -> 25.8 mm, vias 2 -> 3
- net SCL: track 86.8 -> 90.5 mm
- net Net-(AE1-Pad1): track 7.49 -> 4.34 mm
- net Net-(U1-XL1/P0.00): track 5.16 -> 7.39 mm
- net Net-(C5-Pad1): track 0.00 -> 2.01 mm
- net SDA: track 82.8 -> 84.0 mm
- net +3.3V: track 31.1 -> 32.1 mm
- net Net-(U1-XL2/P0.01): track 5.59 -> 4.84 mm, vias 2 -> 0
