File: lightstick_v4/mcu.kicad_sch (KiCad schematic)
At the start: 33 parts, among them J1 FTSH-105-01-F-DV-P-TR, J5 2337019-1, SW1 SW_Push, U1 nRF52840, U5 MX25R6435FZAIL0, U6 AP22814AW5, Y1 32MHz, Y2 32.768kHz

Commit message: rev1
Parts:
- removed J5: 2337019-1, Personal:TE_2337019-1, symbol generic:2337019-1
- added C30: C, Capacitor_SMD:C_0402_1005Metric, symbol Device:C
- added J7: Conn_01x04, Connector_PinHeader_2.54mm:PinHeader_1x04_P2.54mm_Vertical, symbol Connector_Generic:Conn_01x04
- added L2: 2.2nH, Capacitor_SMD:C_0402_1005Metric, symbol Device:L
- C18: LCSC PN C77177 -> C26409; MPN C77177 -> C26409
- Y1: LCSC PN C187794 -> C341819; MPN C187794 -> C341819; Part Number Q22FA12800025 -> Murata XRCGB32M000F2P10R0
- Y2: LCSC PN C32346 -> C97605; MPN C32346 -> C97605; Part Number EPSON Q13FC13500004 -> Seiko SC-32S32.768kHz20PPM9pF
Connections:
- net +3.3V: now also J7.1 (Pin_1)
- net GND: now also C30.2, J7.4 (Pin_4)
- net at C5.1, L1.1: now also L2.2; no longer AE1.1
- net at U1.P2 (P1.08): now also J7.2 (Pin_2)
- net at U1.R1 (TRACEDATA3/P1.09): now also J7.3 (Pin_3)
- new net: AE1.1, C30.1, L2.1
