File: lightstick_v4/power.kicad_sch (KiCad schematic)
At the start: 30 parts, among them J2 USB_C_Receptacle, J6 Conn_01x02, Q1 Q_NMOS_GSD, Q2 Q_NMOS_GSD, Q3 DMG2301L, U3 MCP73831-2-OT, U4 MAX17048, U8 LD39150DT33

Commit message: rev1
Parts:
- D2: LCSC PN C965817 -> C2293; MPN C965817 -> C2293
Changed lines of the file:
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@@
 (kicad_sch
-	(version 20231120)
+	(version 20250114)
 	(generator "eeschema")
-	(generator_version "8.0")
+	(generator_version "9.0")
 	(paper "A4")
 	(junction
@@
 			)
 		)
-		(property "LCSC PN" "C965817"
+		(property "LCSC PN" "C2293"
 			(at 135.89 49.53 90)
 			(effects
@@
 			)
 		)
-		(property "MPN" "C965817"
+		(property "MPN" "C2293"
 			(at 135.89 49.53 90)
 			(effects
